Commit message: Pox implementation of ex1

File: urdf/erl1.urdf (robot description, URDF)
Before this commit: robot erl1, 3 links, 2 joints
Links:
- added link link_arm, mass 1.0; collision box size=1.0 0.05 0.05; visual box size=1.0 0.05 0.05
- added link link_cube, mass 0.3; collision box size=0.1 0.1 0.1; visual box size=0.1 0.1 0.1
Joints:
- added joint arm_joint: type revolute, parent link_cube, child link_arm, origin xyz=0 0 0.1 rpy=0 0 0, axis 0 1 0, limit lower=-3.0 upper=-0.1 effort=5 velocity=1.0
- added joint cube_joint: type revolute, parent link_chassis, child link_cube, origin xyz=0 0 0.035 rpy=0 0 0, axis 0 0 1, limit lower=-1.57 upper=1.57 effort=5 velocity=1.0

Commit message: Camera sensor added

File: urdf/erl1.urdf (robot description, URDF)
Before this commit: robot erl1, 3 links, 2 joints
Links:
- added link camera_link, mass 0.1; collision box size=.03 .03 .03; visual box size=.03 .03 .03
- added link camera_link_optical
Joints:
- added joint camera_joint: type fixed, parent base_link, child camera_link, origin xyz=0.225 0 0.075 rpy=0 0 0, axis 0 1 0
- added joint camera_optical_joint: type fixed, parent camera_link, child camera_link_optical, origin xyz=0 0 0 rpy=-1.5707 0 -1.5707

Commit message: Aligned this repo with the assignment + added lidar

File: urdf/erl1.urdf (robot description, URDF)
Before this commit: robot erl1, 8 links, 7 joints
Links:
- removed link link_chassis
- added link base_footprint
- added link base_link, mass 15.0; collision box size=.4 .2 .1; collision sphere radius=0.0499
- link left_wheel: geometry collision cylinder length=.05 radius=.1; visual mesh filename=package://erl1/meshes/wheel.dae
- link right_wheel: geometry collision cylinder length=.05 radius=.1; visual mesh filename=package://erl1/meshes/wheel.dae
- link scan_link: geometry collision box size=.1 .1 .1; visual mesh filename=package://erl1/meshes/lidar.dae
Joints:
- added joint base_footprint_joint: type fixed, parent base_footprint, child base_link, origin xyz=0 0 0 rpy=0 0 0
- joint left_wheel_joint: origin xyz=-0.1 0.15 0 rpy=0 0 0 -> xyz=0 0.15 0 rpy=0 0 0; parent link_chassis -> base_link
- joint right_wheel_joint: origin xyz=-0.1 -0.15 0 rpy=0 0 0 -> xyz=0 -0.15 0 rpy=0 0 0; parent link_chassis -> base_link
- joint scan_joint: origin (none) -> xyz=0 0 0.15 rpy=0 0 0
